File: design/rev0.brd (EAGLE design)
At the start: 100 x 62 mm, 30 parts, among them U1 CHERRY-MX, U2 CHERRY-MX, U3 CHERRY-MX, U4 CHERRY-MX, U5 CHERRY-MX, U6 CHERRY-MX, U7 CHERRY-MX, U8 CHERRY-MX, U9 CHERRY-MX

Commit message: Add licencing
Other:
- board text added: "Copyright Thomas Pain 2021 This source describes Open Hardware and is licensed under the CERN-OHL-P v2 You may redistribute and modify this documentation and make products using it under the terms of the CERN-OHL-P v2 (https:/cern.ch/cern-ohl). This documentation is distributed WITHOUT ANY EXPRESS OR IMPLIED WARRANTY, INCLUDING OF MERCHANTABILITY, SATISFACTORY QUALITY AND FITNESS FOR A PARTICULAR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"
- board text added: "Licenced under the CERN-OHL-P-2.0 github.com/codemicro/macropad"
Changed lines of the file:
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@@
 Jan 2021</text>
 <text x="49.65" y="26.75" size="1.5" layer="22" font="vector" rot="MR257">001</text>
+<text x="1.6" y="64.95" size="1.778" layer="48">Copyright Thomas Pain 2021
+This source describes Open Hardware and is licensed under the CERN-OHL-P
+v2
+You may redistribute and modify this documentation and make products
+using it under the terms of the CERN-OHL-P v2 (https:/cern.ch/cern-ohl).
+This documentation is distributed WITHOUT ANY EXPRESS OR IMPLIED
+WARRANTY, INCLUDING OF MERCHANTABILITY, SATISFACTORY QUALITY AND FITNESS
+FOR A PARTICULAR PURPOSE. Please see the CERN-OHL-P v2 for applicable
+conditions
+https://github.com/codemicro/macropad</text>
+<text x="92.8" y="56.7" size="1.016" layer="22" rot="MR0">Licenced under the CERN-OHL-P-2.0
+github.com/codemicro/macropad</text>
 </plain>
 <attributes>
