File: design/rev0.sch (EAGLE design)
At the start: 30 parts, among them U1 CHERRY-MX, U2 CHERRY-MX, U3 CHERRY-MX, U4 CHERRY-MX, U5 CHERRY-MX, U6 CHERRY-MX, U7 CHERRY-MX, U8 CHERRY-MX, U9 CHERRY-MX

Commit message: Add licencing
Other:
- note added: "Copyright Thomas Pain 2021 This source describes Open Hardware and is licensed under the CERN-OHL-P v2 You may redistribute and modify this documentation and make products using it under the terms of the CERN-OHL-P v2 (https:/cern.ch/cern-ohl). This documentation is distributed WITHOUT ANY EXPRESS OR IMPLIED WARRANTY, INCLUDING OF MERCHANTABILITY, SATISFACTORY QUALITY AND FITNESS FOR A PARTICULAR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"
Changed lines of the file:
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@@
 <sheet>
 <plain>
+<text x="132.08" y="93.98" size="1.778" layer="97">Copyright Thomas Pain 2021
+This source describes Open Hardware and is licensed under the CERN-OHL-P
+v2
+You may redistribute and modify this documentation and make products
+using it under the terms of the CERN-OHL-P v2 (https:/cern.ch/cern-ohl).
+This documentation is distributed WITHOUT ANY EXPRESS OR IMPLIED
+WARRANTY, INCLUDING OF MERCHANTABILITY, SATISFACTORY QUALITY AND FITNESS
+FOR A PARTICULAR PURPOSE. Please see the CERN-OHL-P v2 for applicable
+conditions
+https://github.com/codemicro/macropad</text>
 </plain>
 <instances>
@@
 </drawing>
 <compatibility>
+<note version="6.3" minversion="6.2.2" severity="warning">
+Since Version 6.2.2 text objects can contain more than one line,
+which will not be processed correctly with this version.
+</note>
 <note version="8.2" severity="warning">
 Since Version 8.2, EAGLE supports online libraries. The ids
